Commit message: Added Project4

File: P4-Map-My-World/my_robot/urdf/my_robot.xacro (robot description, xacro)
@@ -2,4 +2,13 @@
 <robot name="my_robot" xmlns:xacro="http://www.ros.org/wiki/xacro">
   <xacro:include filename="$(find my_robot)/urdf/my_robot.gazebo" />
+  <material name="blue">
+    <color rgba="0 0 0.8 1"/>
+  </material>
+  <material name="black">
+    <color rgba="0 0 0 0"/>
+  </material>
+  <material name="red">
+    <color rgba="0.8 0 0 1"/>
+  </material>
   <link name="robot_footprint"></link>
   <joint name="robot_footprint_joint" type="fixed">
@@ -22,5 +31,5 @@
       <origin xyz="0 0 0" rpy=" 0 0 0"/>
       <geometry>
-        <box size=".4 .4 .1"/>
+        <box size=".45 .25 .15"/>
       </geometry>
     </collision>
@@ -28,37 +37,45 @@
       <origin xyz="0 0 0" rpy=" 0 0 0"/>
       <geometry>
-        <box size=".4 .4 .1"/>
+        <box size=".45 .25 .15"/>
       </geometry>
     </visual>
     <collision name='back_caster_collision'>
-      <origin xyz="-0.15 0 -0.05" rpy=" 0 0 0"/>
-      <geometry>
-        <sphere radius="0.0599"/>
+      <origin xyz="-0.1125 0 -0.075" rpy=" 0 0 0"/>
+      <geometry>
+        <sphere radius="0.0744"/>
       </geometry>
     </collision>
     <visual name='back_caster_visual'>
-      <origin xyz="-0.15 0 -0.05" rpy=" 0 0 0"/>
-      <geometry>
-        <sphere radius="0.0599"/>
+      <origin xyz="-0.1125 0 -0.075" rpy=" 0 0 0"/>
+      <geometry>
+        <sphere radius="0.075"/>
       </geometry>
     </visual>
     <collision name='front_caster_collision'>
-      <origin xyz="0.15 0 -0.05" rpy=" 0 0 0"/>
-      <geometry>
-        <sphere radius="0.0599"/>
+      <origin xyz="0.1125 0 -0.075" rpy=" 0 0 0"/>
+      <geometry>
+        <sphere radius="0.0744"/>
       </geometry>
     </collision>
     <visual name='front_caster_visual'>
-      <origin xyz="0.15 0 -0.05" rpy=" 0 0 0"/>
-      <geometry>
-        <sphere radius="0.0599"/>
-      </geometry>
-    </visual>
-  </link>
-   <link name='left_wheel'>
-    <pose>0 0 0 0 0 0</pose>
-    <inertial>
-      <mass value="5.0"/>
-      <origin xyz="0.0 0 0" rpy=" 0 1.5707 1.5707"/>
+      <origin xyz="0.1125 0 -0.075" rpy=" 0 0 0"/>
+      <geometry>
+        <sphere radius="0.075"/>
+      </geometry>
+    </visual>
+  </link>
+  <gazebo reference="chassis">
+    <material>Gazebo/Red</material>
+  </gazebo>
+  <link name="left_wheel">
+    <collision name='left_wheel'>
+      <origin xyz="0 0 0" rpy=" 0 1.5707 1.5707"/>
+      <geometry>
+        <cylinder radius="0.15" length="0.1"/>
+      </geometry>
+    </collision>
+    <inertial>
+      <mass value="5"/>
+      <origin xyz="0 0 0" rpy=" 0 1.5707 1.5707"/>
       <inertia
           ixx="0.1" ixy="0" ixz="0"
@@ -67,22 +84,21 @@
       />
     </inertial>
-    <collision name='collision'>
-      <origin xyz="0 0 0" rpy=" 0 1.5707 1.5707"/>
-      <geometry>
-        <cylinder radius="0.11" length="0.05"/>
-      </geometry>
-    </collision>
     <visual name='left_wheel_visual'>
       <origin xyz="0 0 0" rpy=" 0 1.5707 1.5707"/>
       <geometry>
-        <cylinder radius="0.11" length="0.05"/>
-      </geometry>
-    </visual>
-  </link>
-   <link name='right_wheel'>
-    <pose>0 0 0 0 0 0</pose>
-    <inertial>
-      <mass value="5.0"/>
-      <origin xyz="0.0 0 0" rpy=" 0 1.5707 1.5707"/>
+        <cylinder radius="0.15" length="0.1"/>
+      </geometry>
+    </visual>
+  </link>
+  <link name="right_wheel">
+    <collision name='right_wheel'>
+      <origin xyz="0 0 0" rpy=" 0 1.5707 1.5707"/>
+      <geometry>
+        <cylinder radius="0.15" length="0.1"/>
+      </geometry>
+    </collision>
+    <inertial>
+      <mass value="5"/>
+      <origin xyz="0 0 0" rpy=" 0 1.5707 1.5707"/>
       <inertia
           ixx="0.1" ixy="0" ixz="0"
@@ -91,19 +107,19 @@
       />
     </inertial>
-    <collision name='collision'>
-      <origin xyz="0 0 0" rpy=" 0 1.5707 1.5707"/>
-      <geometry>
-        <cylinder radius="0.11" length="0.05"/>
-      </geometry>
-    </collision>
     <visual name='right_wheel_visual'>
       <origin xyz="0 0 0" rpy=" 0 1.5707 1.5707"/>
       <geometry>
-        <cylinder radius="0.11" length="0.05"/>
-      </geometry>
-    </visual>
-  </link>
+        <cylinder radius="0.15" length="0.1"/>
+      </geometry>
+    </visual>
+  </link>
+  <gazebo reference="left_wheel">
+    <material>Gazebo/Black</material>
+  </gazebo>
+  <gazebo reference="right_wheel">
+    <material>Gazebo/Black</material>
+  </gazebo>
   <joint type="continuous" name="left_wheel_hinge">
-    <origin xyz="0 0.25 0" rpy="0 0 0"/>
+    <origin xyz="0 0.2 0" rpy="0 0 0"/>
     <child link="left_wheel"/>
     <parent link="chassis"/>
@@ -113,5 +129,5 @@
   </joint>
   <joint type="continuous" name="right_wheel_hinge">
-    <origin xyz="0 -0.25 0" rpy="0 0 0"/>
+    <origin xyz="0 -0.2 0" rpy="0 0 0"/>
     <child link="right_wheel"/>
     <parent link="chassis"/>
@@ -120,9 +136,14 @@
     <dynamics damping="1.0" friction="1.0"/>
   </joint>
- <link name='camera'>
-    <pose>0 0 0 0 0 0</pose>
+  <link name="camera">
+    <collison name="camera">
+      <origin xyz="0 0 0" rpy="0 0 0"/>
+      <geometry>
+        <box size="0.05 0.05 0.05"/>
+      </geometry>
+    </collison>
     <inertial>
       <mass value="0.1"/>
-      <origin xyz="0.0 0 0" rpy="0.0 0 0"/>
+      <origin xyz="0 0 0" rpy="0 0 0"/>
       <inertia
           ixx="1e-6" ixy="0" ixz="0"
@@ -131,38 +152,30 @@
       />
     </inertial>
-    <collision name='collision'>
-      <origin xyz="0 0 0" rpy="0.0 0 0"/>
+    <visual name="camera">
+      <origin xyz="0 0 0" rpy="0 0 0"/>
       <geometry>
         <box size="0.05 0.05 0.05"/>
       </geometry>
-    </collision>
-    <visual name='camera_visual'>
-      <origin xyz="0.0 0 0" rpy="0.0 0 0"/>
-      <geometry>
-        <box size="0.05 0.05 0.05"/>
-      </geometry>
-    </visual>
+    </visual>
+    <box_inertia sizeX="0.05" sizeY="0.05" sizeZ="0.05" mass="0.1">
+      <origin xyz="0 0 0" rpy="0 0 0" />
+    </box_inertia>
   </link>
   <joint type="fixed" name="camera_joint">
-    <origin xyz="0.2 0 0" rpy="0 0 0"/>
+    <origin xyz="0.225 0 0" rpy="0 0 0"/>
     <child link="camera"/>
     <parent link="chassis"/>
-    <axis xyz="0 1 0" rpy="0 0 0"/>
-    <limit effort="10000" velocity="1000"/>
-    <dynamics damping="1.0" friction="1.0"/>
-  </joint>
-    <!-- RGB-D camera -->
-    <joint type="fixed" name="camera_optical_joint">
-      <origin xyz="0 0 0" rpy="-1.5707 0 -1.5707"/>
-      <parent link="camera"/>
-      <child link="camera_optical"/>
-    </joint>
-    <link name="camera_optical">
-    </link>
- <link name='hokuyo'>
-    <pose>0 0 0 0 0 0</pose>
+    <axis xyz="0 1 0"/>
+  </joint>
+  <link name="hokuyo">
+    <collison name="hokuyo">
+      <origin xyz="0 0 0" rpy="0 0 0"/>
+      <geometry>
+        <box size="0.1 0.1 0.1"/>
+      </geometry>
+    </collison>
     <inertial>
       <mass value="1e-5"/>
-      <origin xyz="0.0 0 0" rpy="0.0 0 0"/>
+      <origin xyz="0 0 0" rpy="0 0 0"/>
       <inertia
           ixx="1e-6" ixy="0" ixz="0"
@@ -171,14 +184,8 @@
       />
     </inertial>
-    <collision name='collision'>
-      <origin xyz="0 0 0" rpy="0.0 0 0"/>
-      <geometry>
-	<box size="0.1 0.1 0.1"/>
-      </geometry>
-    </collision>
-    <visual name='hokuyo_visual'>
-      <origin xyz="0.0 0 0" rpy="0.0 0 0"/>
-      <geometry>
-	<mesh filename="package://my_robot/meshes/hokuyo.dae"/>
+    <visual name="hokuyo">
+      <origin xyz="0 0 0" rpy="0 0 0"/>
+      <geometry>
+        <mesh filename = "package://my_robot/meshes/hokuyo.dae"/>
       </geometry>
     </visual>
@@ -188,19 +195,12 @@
     <child link="hokuyo"/>
     <parent link="chassis"/>
-    <axis xyz="0 1 0" rpy="0 0 0"/>
-    <limit effort="10000" velocity="1000"/>
-    <dynamics damping="1.0" friction="1.0"/>
-  </joint>
-  <gazebo reference="left_wheel">
-    <material>Gazebo/Red</material>
-  </gazebo>
-  <gazebo reference="right_wheel">
-    <material>Gazebo/Red</material>
-  </gazebo>
-  <gazebo reference="chassis">
-    <material>Gazebo/Blue</material>
-  </gazebo>
-  <gazebo reference="camera">
-    <material>Gazebo/Green</material>
-  </gazebo>
+    <axis xyz="0 1 0"/>
+  </joint>
+  <joint name="camera_optical_joint" type="fixed">
+    <origin xyz="0 0 0" rpy="-1.5707 0 -1.5707"/>
+    <parent link="camera"/>
+    <child link="camera_link_optical"/>
+  </joint>
+  <link name="camera_link_optical">
+  </link>
 </robot>
